Commit message: feat(core): synchronize mobile robot masterclass with navigation architecture
- Kinematics & Skid-Steer Tuning: Calibrate effective track width (0.457m Classic, 0.380m Ignition) in controller params and Gazebo plugins.
- REP-103 Optical Frames: Add standard camera_optical_link frame and Ignition IMU sensor definition.
- Smart Telemetry Bridge: Implement auto-sensing discriminator for SI vs raw ADC counts in serial bridge.
- C++ Firmware Declarations: Add function prototypes and ESP32 Core 2.x/3.x LEDC macro guards.
- Safety Zone Controller: Add dynamic /safety_zone_enable bypass topic and clean state-change logging.
- Decoupled Launchers: Cleanly separate ros2_control vs custom kinematics controllers and add simulation worlds.
- Universal Portability: Dynamically resolve WS_DIR across all verification scripts and automation tools.

File: src/mobile_robot_description/urdf/mobile_robot.urdf.xacro (robot description, xacro)
@@ -263,4 +263,11 @@
     <origin xyz="0.20 0.0 0.05" rpy="0 0 0"/>
   </joint>
+  <!-- Standard ROS Camera Optical Frame (Z forward, X right, Y down) -->
+  <link name="camera_optical_link"/>
+  <joint name="camera_optical_joint" type="fixed">
+    <parent link="camera_link"/>
+    <child link="camera_optical_link"/>
+    <origin xyz="0 0 0" rpy="${-PI/2} 0 ${-PI/2}"/>
+  </joint>
   <!-- 7C. IMU Sensor Link (MPU6050 / BNO055 Breakout Board) -->
   <link name="imu_link">

File: src/mobile_robot_description/urdf/mobile_robot_gazebo.xacro (robot description, xacro)
@@ -34,5 +34,5 @@
   <!-- ==================================================================== -->
   <xacro:arg name="is_ignition" default="false"/>
-  <xacro:arg name="use_ros2_control" default="true"/>
+  <xacro:arg name="use_ros2_control" default="false"/>
   <!-- ==================================================================== -->
   <!-- 2A. GAZEBO CLASSIC (Gazebo 11) PLUGINS (Only when NOT Ignition)      -->
@@ -69,13 +69,13 @@
           <right_joint>front_right_wheel_joint</right_joint>
           <right_joint>rear_right_wheel_joint</right_joint>
-          <!-- Kinematics -->
-          <wheel_separation>0.34</wheel_separation>
+          <!-- Kinematics (Calibrated for 4WD skid-steer wheel scrub) -->
+          <wheel_separation>0.457</wheel_separation>
           <wheel_diameter>0.10</wheel_diameter>
           <!-- Limits -->
           <max_wheel_torque>20.0</max_wheel_torque>
           <max_wheel_acceleration>2.0</max_wheel_acceleration>
-          <!-- Output / Odometry (Handled by diff_drive_controller) -->
-          <publish_odom>false</publish_odom>
-          <publish_odom_tf>false</publish_odom_tf>
+          <!-- Output / Odometry (Handled by Gazebo diff drive plugin) -->
+          <publish_odom>true</publish_odom>
+          <publish_odom_tf>true</publish_odom_tf>
           <publish_wheel_tf>false</publish_wheel_tf>
           <odometry_frame>odom</odometry_frame>
@@ -115,6 +115,6 @@
           </scan>
           <range>
-            <min>0.08</min>
-            <max>10.0</max>
+            <min>0.15</min>
+            <max>12.0</max>
             <resolution>0.01</resolution>
           </range>
@@ -132,5 +132,5 @@
     <gazebo reference="camera_link">
       <sensor name="front_camera" type="camera">
-        <pose>0 0 0 0 0 0</pose>
+        <pose>0.021 0 0 0 0 0</pose>
         <always_on>true</always_on>
         <visualize>false</visualize>
@@ -144,15 +144,16 @@
           </image>
           <clip>
-            <near>0.05</near>
-            <far>8.0</far>
+            <near>0.02</near>
+            <far>12.0</far>
           </clip>
         </camera>
         <plugin name="camera_controller" filename="libgazebo_ros_camera.so">
           <ros>
+            <namespace>/</namespace>
             <remapping>~/image_raw:=/camera/image_raw</remapping>
             <remapping>~/camera_info:=/camera/camera_info</remapping>
           </ros>
           <camera_name>camera</camera_name>
-          <frame_name>camera_link</frame_name>
+          <frame_name>camera_optical_link</frame_name>
         </plugin>
       </sensor>
@@ -193,5 +194,5 @@
       </xacro:if>
       <xacro:unless value="$(arg use_ros2_control)">
-        <!-- Option A - Diff Drive System for Ignition / Modern Gazebo -->
+        <!-- Option A - Diff Drive System for Ignition / Modern Gazebo (Calibrated for Ignition/Gz DART physics) -->
         <plugin filename="libignition-gazebo-diff-drive-system.so" name="ignition::gazebo::systems::DiffDrive">
           <left_joint>front_left_wheel_joint</left_joint>
@@ -199,7 +200,6 @@
           <right_joint>front_right_wheel_joint</right_joint>
           <right_joint>rear_right_wheel_joint</right_joint>
-          <wheel_separation>0.34</wheel_separation>
+          <wheel_separation>0.380</wheel_separation>
           <wheel_radius>0.05</wheel_radius>
-          <odom_publish_frequency>50</odom_publish_frequency>
           <topic>/cmd_vel</topic>
           <odom_topic>/odom</odom_topic>
@@ -207,18 +207,27 @@
           <frame_id>odom</frame_id>
           <child_frame_id>base_footprint</child_frame_id>
+          <odom_publish_frequency>50</odom_publish_frequency>
+        </plugin>
+        <!-- Joint State Publisher for Ignition / Modern Gazebo (Only when NOT using ros2_control) -->
+        <plugin filename="libignition-gazebo-joint-state-publisher-system.so" name="ignition::gazebo::systems::JointStatePublisher">
+          <topic>/joint_states</topic>
+          <update_rate>50.0</update_rate>
+          <joint_name>front_left_wheel_joint</joint_name>
+          <joint_name>front_right_wheel_joint</joint_name>
+          <joint_name>rear_left_wheel_joint</joint_name>
+          <joint_name>rear_right_wheel_joint</joint_name>
         </plugin>
       </xacro:unless>
-      <!-- Joint State Publisher for Ignition / Modern Gazebo -->
-      <plugin filename="libignition-gazebo-joint-state-publisher-system.so" name="ignition::gazebo::systems::JointStatePublisher">
-        <topic>/joint_states</topic>
-      </plugin>
-      <!-- Sensors System for Ignition / Modern Gazebo -->
-      <plugin filename="libignition-gazebo-sensors-system.so" name="ignition::gazebo::systems::Sensors">
-        <render_engine>ogre2</render_engine>
-      </plugin>
-      <!-- IMU System for Ignition / Modern Gazebo -->
-      <plugin filename="libignition-gazebo-imu-system.so" name="ignition::gazebo::systems::Imu"/>
     </gazebo>
     <!-- Ignition / Modern Gz Sensors -->
+    <gazebo reference="imu_link">
+      <sensor name="imu_sensor" type="imu">
+        <always_on>1</always_on>
+        <update_rate>50.0</update_rate>
+        <visualize>false</visualize>
+        <topic>/imu/data</topic>
+        <gz_frame_id>imu_link</gz_frame_id>
+      </sensor>
+    </gazebo>
     <gazebo reference="lidar_link">
       <sensor name="lidar_sensor_ign" type="gpu_lidar">
@@ -239,6 +248,6 @@
           </scan>
           <range>
-            <min>0.08</min>
-            <max>10.0</max>
+            <min>0.15</min>
+            <max>12.0</max>
             <resolution>0.01</resolution>
           </range>
@@ -248,10 +257,10 @@
     <gazebo reference="camera_link">
       <sensor name="front_camera_ign" type="camera">
-        <pose>0 0 0 0 0 0</pose>
+        <pose>0.021 0 0 0 0 0</pose>
         <always_on>true</always_on>
         <visualize>false</visualize>
         <update_rate>30.0</update_rate>
         <topic>/camera/image_raw</topic>
-        <gz_frame_id>camera_link</gz_frame_id>
+        <gz_frame_id>camera_optical_link</gz_frame_id>
         <camera>
           <horizontal_fov>1.089</horizontal_fov>
@@ -262,6 +271,6 @@
           </image>
           <clip>
-            <near>0.05</near>
-            <far>8.0</far>
+            <near>0.02</near>
+            <far>12.0</far>
           </clip>
         </camera>
